Commit message: simplified collision geometry of fingers

File: yumi_description/urdf/yumi_servo_gripper.xacro (robot description, xacro)
@@ -68,7 +68,8 @@
       </visual>
       <collision>
-        <origin xyz="0 0 0" rpy="0 0 0"/>
+        <origin xyz="-0.005 0.005 0" rpy="0 0 0"/>
         <geometry>
-          <mesh filename="package://yumi_description/meshes/gripper/coarse/finger.stl"/>
+          <cylinder length="0.1" radius="0.005"/>
+          <!--mesh filename="package://yumi_description/meshes/gripper/coarse/finger.stl"/-->
         </geometry>
         <material name="Grey"/>
@@ -104,7 +105,8 @@
       </visual>
       <collision>
-        <origin xyz="0 0 0" rpy="0 0 0"/>
+        <origin xyz="-0.005 0.005 0" rpy="0 0 0"/>
         <geometry>
-          <mesh filename="package://yumi_description/meshes/gripper/coarse/finger.stl"/>
+          <cylinder length="0.1" radius="0.005"/>
+          <!--mesh filename="package://yumi_description/meshes/gripper/coarse/finger.stl"/-->
         </geometry>
         <material name="Grey"/>

Commit message: add spring damper to joints

File: yumi_description/urdf/yumi_servo_gripper.xacro (robot description, xacro)
@@ -8,5 +8,5 @@
   <xacro:include filename="$(find yumi_description)/urdf/utilities.xacro" />
   <!-- some constants -->
- <!-- <xacro:property name="safety_controller_k_pos" value="100" />
+  <!-- <xacro:property name="safety_controller_k_pos" value="100" />
   <xacro:property name="safety_controller_k_vel" value="2" /> -->
   <xacro:property name="joint_damping" value="0.5" />
@@ -47,5 +47,5 @@
       <axis xyz="-1 0 0"/>
       <limit lower="0" upper="0.025"
-             effort="${max_effort}" velocity="0.02" />
+        effort="${max_effort}" velocity="0.02" />
       <!--   <safety_controller soft_lower_limit="${-168 * M_PI / 180}"
            soft_upper_limit="${168 * M_PI / 180}"
@@ -54,4 +54,10 @@
       <dynamics damping="${joint_damping}"/>
     </joint>
+    <gazebo reference="${name}_joint">
+      <implicitSpringDamper>1</implicitSpringDamper>
+    </gazebo>
+    <gazebo reference="${name}_joint_m">
+      <implicitSpringDamper>1</implicitSpringDamper>
+    </gazebo>
     <link name="${name}_finger_r">
       <inertial>
@@ -75,5 +81,5 @@
       </collision>
     </link>
-   <!-- joint between base and left finger -->
+    <!-- joint between base and left finger -->
     <joint name="${name}_joint_m" type="prismatic">
       <parent link="${name}_base"/>
@@ -82,5 +88,5 @@
       <axis xyz="-1 0 0"/>
       <limit lower="0" upper="0.025"
-             effort="${max_effort}" velocity="0.02" />
+        effort="${max_effort}" velocity="0.02" />
       <!--   <safety_controller soft_lower_limit="${-168 * M_PI / 180}"
            soft_upper_limit="${168 * M_PI / 180}"
@@ -111,5 +117,5 @@
       </collision>
     </link>
-     <!--Extensions -->
+    <!--Extensions -->
     <xacro:yumi_servo_gripper_gazebo name="${name}" />
     <xacro:yumi_servo_gripper_transmission name="${name}" hardware_interface="hardware_interface/${hardware_interface}"/>

Commit message: add contact info + make gripper bigger

File: yumi_description/urdf/yumi_servo_gripper.xacro (robot description, xacro)
@@ -61,4 +61,9 @@
     </gazebo>
     <link name="${name}_finger_r">
+      <contact>
+        <lateral_friction value="1.0"/>
+        <spinning_friction value="1.5"/>
+        <inertia_scaling value="0.3"/>
+      </contact>
       <inertial>
         <origin xyz="0 0 0" rpy="0 0 0"/>
@@ -76,5 +81,6 @@
         <origin xyz="-0.005 0.005 0" rpy="0 0 0"/>
         <geometry>
-          <cylinder length="0.1" radius="0.005"/>
+          <box size="0.005 0.01 0.1"/>
+          <!--cylinder length="0.1" radius="0.005"/-->
           <!--mesh filename="package://yumi_description/meshes/gripper/coarse/finger.stl"/-->
         </geometry>
@@ -98,4 +104,9 @@
     </joint>
     <link name="${name}_finger_l">
+      <contact>
+        <lateral_friction value="1.0"/>
+        <spinning_friction value="1.5"/>
+        <inertia_scaling value="0.3"/>
+      </contact>
       <inertial>
         <origin xyz="0 0 0" rpy="0 0 0"/>
@@ -113,5 +124,6 @@
         <origin xyz="-0.005 0.005 0" rpy="0 0 0"/>
         <geometry>
-          <cylinder length="0.1" radius="0.005"/>
+          <box size="0.025 0.015 0.1"/>
+          <!--cylinder length="0.1" radius="0.005"/-->
           <!--mesh filename="package://yumi_description/meshes/gripper/coarse/finger.stl"/-->
         </geometry>

Commit message: bigger gripper

File: yumi_description/urdf/yumi_servo_gripper.xacro (robot description, xacro)
@@ -81,5 +81,5 @@
         <origin xyz="-0.005 0.005 0" rpy="0 0 0"/>
         <geometry>
-          <box size="0.005 0.01 0.1"/>
+          <box size="0.01 0.012 0.1"/>
           <!--cylinder length="0.1" radius="0.005"/-->
           <!--mesh filename="package://yumi_description/meshes/gripper/coarse/finger.stl"/-->
@@ -124,5 +124,5 @@
         <origin xyz="-0.005 0.005 0" rpy="0 0 0"/>
         <geometry>
-          <box size="0.025 0.015 0.1"/>
+          <box size="0.01 0.012 0.1"/>
           <!--cylinder length="0.1" radius="0.005"/-->
           <!--mesh filename="package://yumi_description/meshes/gripper/coarse/finger.stl"/-->
